File: electronics/Lamp.kicad_pcb (KiCad board)
At the start: 2 copper layers, 67.4 x 28.6 mm, 26 parts, among them J1 USB_A, J2 USB_A, Q1 2N7002, Q2 AO3401A, Q3 2N7002, Q4 AO3401A, Q5 AO3400A, SW1 SW_Push, SW2 SW_Push, U1 ESP32-C6_SUPERMINI_SMD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

Commit message: Update PCB
Parts:
- moved U1 0.25 mm to (162.0, 137.5)
Routing:
- net GND: track 128.6 -> 0.00 mm, vias 3 -> 0
- net +5V: track 88.9 -> 0.00 mm, vias 3 -> 0
- net Net-(Q3-G): track 31.7 -> 0.00 mm
- net Net-(U1-GPIO6): track 31.0 -> 0.00 mm
- net Net-(Q1-G): track 25.8 -> 0.00 mm
- net /Clim: track 24.5 -> 0.00 mm, vias 1 -> 0
- net Net-(U1-GPIO3): track 20.9 -> 0.00 mm
- net Net-(U1-GPIO14): track 14.9 -> 0.00 mm
- net /Sheild: track 13.2 -> 0.00 mm
- net Net-(U2B--): track 9.58 -> 0.00 mm
- net Net-(Q5-G): track 6.55 -> 0.00 mm, vias 1 -> 0
- net Net-(Q3-D): track 6.42 -> 0.00 mm
- net Net-(Q1-D): track 6.38 -> 0.00 mm
- net Net-(U2A-+): track 5.27 -> 0.00 mm
- net Net-(Q5-S): track 4.13 -> 0.00 mm, vias 1 -> 0
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