File: electronics/Lamp.kicad_sch (KiCad schematic)
At the start: 24 parts, among them J1 USB_A, J2 USB_A, Q1 2N7002, Q2 AO3401A, Q3 2N7002, Q4 AO3401A, Q5 AO3400A, SW1 SW_Push, SW2 SW_Push, U1 ESP32-C6_SUPERMINI_SMD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

Commit message: WIP the schematic
Parts:
- added J3: USB_C_Receptacle_PowerOnly_6P, symbol Connector:USB_C_Receptacle_PowerOnly_6P
- added R12: 4.7K, Resistor_SMD:R_0805_2012Metric_Pad1.20x1.40mm_HandSolder, symbol Device:R
- R11: value 10K -> 4.7K
Connections:
- net +5V: no longer C2.1, R11.1, U2.8 (V+)
- net at U1.6 (GPIO6), U2.7: now also R12.2
- net +3V3: now reaches U1.3.3 (3V3)
- net +3V3: now also C2.1, R11.1, U2.8 (V+), R12.1
- new net: J3.A12 (GND), J3.B12 (GND)
- new net: J3.A9 (VBUS), J3.B9 (VBUS)
- no-connect marks 17 -> 16
Other:
- moved on the sheet: R11

Commit message: Update schamatic
Parts:
- removed J3: USB_C_Receptacle_PowerOnly_6P, symbol Connector:USB_C_Receptacle_PowerOnly_6P
- added C3: C, symbol Device:C
- added J4: USB_C_Receptacle_USB2.0_14P, Connector_USB:USB_C_Receptacle_GCT_USB4110, symbol Connector:USB_C_Receptacle_USB2.0_14P
- added R13: 10K, symbol Device:R
- added R14: 1K, symbol Device:R
- added U3: CH224K, Package_SO:SSOP-10-1EP_3.9x4.9mm_P1mm_EP2.1x3.3mm, symbol Interface_USB:CH224K
Connections:
- net GND: now also C3.2, U3.11 (GND)
- new net: C3.1, R14.1, U3.1 (VDD)
- new net: R13.1, U3.8 (VBUS)
- new net: J4.A6 (D+), J4.B6 (D+), U3.4 (DP)
- new net: J4.A7 (D-), J4.B7 (D-), U3.5 (DM)
- new net: J4.A5 (CC1), U3.6 (CC2)
- new net: J4.B5 (CC2), U3.7 (CC1)
- new net: J4.A1 (GND), J4.A12 (GND), J4.B1 (GND), J4.B12 (GND)
- new net: J4.A4 (VBUS), J4.A9 (VBUS), J4.B4 (VBUS), J4.B9 (VBUS)
